File: PCBs/ConnsBoard/Kicad_minisumo_up.kicad_pcb (KiCad board)
At the start: 2 copper layers, 92 x 32 mm, 41 parts, among them J1 Screw_Terminal_01x15, J13 screw, J14 screw, J15 screw, J2 Screw_Terminal_01x17, M2 MountingHole_2.2mm_M2

Commit message: Rotate supply connector to match supply wires colors
Parts:
- moved S-11.1V 1.19 mm to (131.3, 57.8), turned to 180 degrees
Routing:
- net +11.1V: track 8.66 -> 14.3 mm
Changed lines of the file:
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@@
 	(footprint "Connector_JST:JST_PH_B2B-PH-K_1x02_P2.00mm_Vertical"
 		(layer "F.Cu")
-		(at 130.9 56.71)
+		(at 131.33 57.82 180)
 		(descr "JST PH series connector, B2B-PH-K (http://www.jst-mfg.com/product/pdf/eng/ePH.pdf), generated with kicad-footprint-generator")
 		(tags "connector JST PH side entry")
 		(property "Reference" "S-11.1V"
-			(at -3.3 0.59 90)
+			(at 5.28 0.55 90)
 			(layer "F.SilkS")
 			(effects
@@
 		)
 		(property "Datasheet" ""
-			(at 0 0 0)
+			(at 0 0 180)
 			(unlocked yes)
 			(layer "F.Fab")
@@
 		)
 		(property "Description" "Generic screw terminal, single row, 01x02, script generated (kicad-library-utils/schlib/autogen/connector/)"
-			(at 0 0 0)
+			(at 0 0 180)
 			(unlocked yes)
 			(layer "F.Fab")
@@
 		(attr through_hole)
 		(fp_line
-			(start -2.36 -2.11)
-			(end -2.36 -0.86)
+			(start 4.06 2.91)
+			(end 4.06 -1.81)
 			(stroke
 				(width 0.12)
@@
 		)
 		(fp_line
-			(start -2.06 -1.81)
-			(end -2.06 2.91)
+			(start 4.06 0.8)
+			(end 3.45 0.8)
 			(stroke
 				(width 0.12)
@@
 		)
 		(fp_line
-			(start -2.06 -0.5)
-			(end -1.45 -0.5)
+			(start 4.06 -0.5)
+			(end 3.45 -0.5)
 			(stroke
 				(width 0.12)
@@
 		)
 		(fp_line
-			(start -2.06 0.8)
-			(end -1.45 0.8)
+			(start 4.06 -1.81)
+			(end -2.06 -1.81)
 			(stroke
 				(width 0.12)
@@
 		)
 		(fp_line
-			(start -2.06 2.91)
-			(end 4.06 2.91)
+			(start 3.45 2.3)
+			(end 3.45 -1.2)
 			(stroke
 				(width 0.12)
@@
 		)
 		(fp_line
-			(start -1.45 -1.2)
-			(end -1.45 2.3)
+			(start 3.45 -1.2)
+			(end 1.5 -1.2)
 			(stroke
 				(width 0.12)
@@
 		)
 		(fp_line
-			(start -1.45 2.3)
-			(end 3.45 2.3)
+			(start 1.5 -1.2)
+			(end 1.5 -1.81)
 			(stroke
 				(width 0.12)
@@
 		)
 		(fp_line
-			(start -1.11 -2.11)
-			(end -2.36 -2.11)
+			(start 1.1 1.8)
+			(end 1.1 2.3)
 			(stroke
 				(width 0.12)
@@
 		)
 		(fp_line
-			(start -0.6 -2.01)
-			(end -0.6 -1.81)
+			(start 1 2.3)
+			(end 1 1.8)
 			(stroke
 				(width 0.12)
@@
 		)
 		(fp_line
-			(start -0.3 -2.01)
-			(end -0.6 -2.01)
+			(start 0.9 2.3)
+			(end 0.9 1.8)
 			(stroke
 				(width 0.12)
@@
 		)
 		(fp_line
-			(start -0.3 -1.91)
-			(end -0.6 -1.91)
+			(start 0.9 1.8)
+			(end 1.1 1.8)
 			(stroke
 				(width 0.12)
@@
 		)
 		(fp_line
-			(start -0.3 -1.81)
-			(end -0.3 -2.01)
+			(start 0.5 -1.2)
+			(end -1.45 -1.2)
 			(stroke
 				(width 0.12)
@@
 		)
 		(fp_line
-			(start 0.5 -1.2)
-			(end -1.45 -1.2)
+			(start -0.3 -1.81)
+			(end -0.3 -2.01)
 			(stroke
 				(width 0.12)
@@
 		)
 		(fp_line
-			(start 0.9 1.8)
-			(end 1.1 1.8)
+			(start -0.3 -1.91)
+			(end -0.6 -1.91)
 			(stroke
 				(width 0.12)
@@
 		)
 		(fp_line
-			(start 0.9 2.3)
-			(end 0.9 1.8)
+			(start -0.3 -2.01)
+			(end -0.6 -2.01)
 			(stroke
 				(width 0.12)
@@
 		)
 		(fp_line
-			(start 1 2.3)
-			(end 1 1.8)
+			(start -0.6 -2.01)
+			(end -0.6 -1.81)
 			(stroke
 				(width 0.12)
@@
 		)
 		(fp_line
-			(start 1.1 1.8)
-			(end 1.1 2.3)
+			(start -1.11 -2.11)
+			(end -2.36 -2.11)
 			(stroke
 				(width 0.12)
@@
 		)
 		(fp_line
-			(start 1.5 -1.2)
-			(end 1.5 -1.81)
+			(start -1.45 2.3)
+			(end 3.45 2.3)
 			(stroke
 				(width 0.12)
@@
 		)
 		(fp_line
-			(start 3.45 -1.2)
-			(end 1.5 -1.2)
+			(start -1.45 -1.2)
+			(end -1.45 2.3)
 			(stroke
 				(width 0.12)
@@
 		)
 		(fp_line
-			(start 3.45 2.3)
-			(end 3.45 -1.2)
+			(start -2.06 2.91)
+			(end 4.06 2.91)
 			(stroke
 				(width 0.12)
@@
 		)
 		(fp_line
-			(start 4.06 -1.81)
-			(end -2.06 -1.81)
+			(start -2.06 0.8)
+			(end -1.45 0.8)
 			(stroke
 				(width 0.12)
@@
 		)
 		(fp_line
-			(start 4.06 -0.5)
-			(end 3.45 -0.5)
+			(start -2.06 -0.5)
+			(end -1.45 -0.5)
 			(stroke
 				(width 0.12)
@@
 		)
 		(fp_line
-			(start 4.06 0.8)
-			(end 3.45 0.8)
+			(start -2.06 -1.81)
+			(end -2.06 2.91)
 			(stroke
 				(width 0.12)
@@
 		)
 		(fp_line
-			(start 4.06 2.91)
-			(end 4.06 -1.81)
+			(start -2.36 -2.11)
+			(end -2.36 -0.86)
 			(stroke
 				(width 0.12)
@@
 		)
 		(fp_line
-			(start -2.45 -2.2)
-			(end -2.45 3.3)
+			(start 4.45 3.3)
+			(end 4.45 -2.2)
 			(stroke
 				(width 0.05)
@@
 		)
 		(fp_line
-			(start -2.45 3.3)
-			(end 4.45 3.3)
+			(start 4.45 -2.2)
+			(end -2.45 -2.2)
 			(stroke
 				(width 0.05)
@@
 		)
 		(fp_line
-			(start 4.45 -2.2)
-			(end -2.45 -2.2)
+			(start -2.45 3.3)
+			(end 4.45 3.3)
 			(stroke
 				(width 0.05)
@@
 		)
 		(fp_line
-			(start 4.45 3.3)
-			(end 4.45 -2.2)
+			(start -2.45 -2.2)
+			(end -2.45 3.3)
 			(stroke
 				(width 0.05)
@@
 		)
 		(fp_line
-			(start -2.36 -2.11)
-			(end -2.36 -0.86)
+			(start 3.95 2.8)
+			(end 3.95 -1.7)
 			(stroke
 				(width 0.1)
@@
 		)
 		(fp_line
-			(start -1.95 -1.7)
-			(end -1.95 2.8)
+			(start 3.95 -1.7)
+			(end -1.95 -1.7)
 			(stroke
 				(width 0.1)
@@
 		)
 		(fp_line
-			(start -1.95 2.8)
-			(end 3.95 2.8)
+			(start -1.11 -2.11)
+			(end -2.36 -2.11)
 			(stroke
 				(width 0.1)
@@
 		)
 		(fp_line
-			(start -1.11 -2.11)
-			(end -2.36 -2.11)
+			(start -1.95 2.8)
+			(end 3.95 2.8)
 			(stroke
 				(width 0.1)
@@
 		)
 		(fp_line
-			(start 3.95 -1.7)
-			(end -1.95 -1.7)
+			(start -1.95 -1.7)
+			(end -1.95 2.8)
 			(stroke
 				(width 0.1)
@@
 		)
 		(fp_line
-			(start 3.95 2.8)
-			(end 3.95 -1.7)
+			(start -2.36 -2.11)
+			(end -2.36 -0.86)
 			(stroke
 				(width 0.1)
@@
 		)
 		(pad "1" thru_hole roundrect
-			(at 0 0)
+			(at 0 0 180)
 			(size 1.2 1.75)
 			(drill 0.75)
@@
 		)
 		(pad "2" thru_hole oval
-			(at 2 0)
+			(at 2 0 180)
 			(size 1.2 1.75)
 			(drill 0.75)
@@
 	)
 	(segment
-		(start 136.76 58.2)
-		(end 135.27 56.71)
+		(start 130.31 55.62)
+		(end 129.33 56.6)
 		(width 1.3)
 		(layer "F.Cu")
@@
 	)
 	(segment
-		(start 135.27 56.71)
-		(end 132.9 56.71)
+		(start 138.4 58.2)
+		(end 136.76 58.2)
 		(width 1.3)
 		(layer "F.Cu")
@@
 	)
 	(segment
-		(start 138.4 58.2)
-		(end 136.76 58.2)
+		(start 134.18 55.62)
+		(end 130.31 55.62)
+		(width 1.3)
+		(layer "F.Cu")
+		(net 28)
+	)
+	(segment
+		(start 136.76 58.2)
+		(end 134.18 55.62)
+		(width 1.3)
+		(layer "F.Cu")
+		(net 28)
+	)
+	(segment
+		(start 129.33 56.6)
+		(end 129.33 57.82)
 		(width 1.3)
 		(layer "F.Cu")
