File: PCBs/MainBoard/Kicad_MiniSumo.kicad_pcb (KiCad board)
At the start: 2 copper layers, 92 x 32 mm, 18 parts, among them J1 Screw_Terminal_01x15, M2 MountingHole_2.2mm_M2

Commit message: fix: remove already fixed comments
Other:
- board text removed: "CHANGE PADS TO THERMAL RELEASES IN NEXT VERSION!!!"
- board text removed: "MAKE BIGGER THTs (to the size of STM one)"
Changed lines of the file:
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@@
-		)
-	)
-	(gr_text "CHANGE PADS TO THERMAL RELEASES IN NEXT VERSION!!!"
-		(at 130.556 62.103 0)
-		(layer "F.Fab")
-		(effects
-			(font
-				(size 1.5 1.5)
-				(thickness 0.3)
-				(bold yes)
-			)
-			(justify left bottom)
 		)
 	)
@@
 		)
 	)
-	(gr_text "MAKE BIGGER THTs (to the size of STM one)"
-		(at 136.398 55.753 0)
+	(gr_text "REMOVE CN16 ON NUCLEO BOARD BEFORE SOLDIERING"
+		(at 131.99 62.66 0)
 		(layer "F.Fab")
 		(effects
-			(font
-				(size 1.5 1.5)
-				(thickness 0.3)
-				(bold yes)
-			)
-			(justify left bottom)
-		)
-	)
-	(gr_text "REMOVE CN16 ON NUCLEO BOARD BEFORE SOLDIERING"
-		(at 131.572 59.055 0)
-		(layer "F.Fab")
-		(effects

Commit message: fix: add comment about changing the uC
Other:
- board text added: "Change Nucleo into a normal STM32 and give NORMAL PWM to the motors"
Changed lines of the file:
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@@
+		)
+	)
+	(gr_text "Change Nucleo into a normal STM32 and give NORMAL PWM to the motors"
+		(at 122.12 59.82 0)
+		(layer "F.Fab")
+		(effects
+			(font
+				(size 1.5 1.5)
+				(thickness 0.3)
+				(bold yes)
+			)
+			(justify left bottom)
 		)
 	)
